File: kicad/pedal_kicad.kicad_sch (KiCad schematic)
At the start: 9 parts

Commit message: new sheet
Parts:
- removed C10, C15: 100n, symbol Device:C
- removed C11, C12, C13, C14: 220u, symbol Device:C
- removed R13, R14: 300, symbol Device:R
- removed TP4: 3V3 TP, symbol Connector:TestPoint
Other:
- added sheet power_supply (power_supply.kicad_sch)

Commit message: power suply done
Changed lines of the file:
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@@
 	(paper "A4")
 	(sheet
-		(at 31.75 25.4)
-		(size 80.01 87.63)
-		(fields_autoplaced yes)
+		(at 13.97 21.59)
+		(size 62.23 58.42)
 		(stroke
 			(width 0.1524)
@@
 		)
 		(property "Sheetname" "power_supply"
-			(at 31.75 24.6884 0)
+			(at 14.224 20.828 0)
 			(effects
 				(font
@@
 		)
 		(property "Sheetfile" "power_supply.kicad_sch"
-			(at 31.75 113.6146 0)
+			(at 13.97 109.8046 0)
 			(effects
 				(font

Commit message: commit a crime
Other:
- added sheet Switches, Buttons, LED (switchesButtonsLed.kicad_sch)
Changed lines of the file:
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@@
 	(paper "A4")
+	(sheet
+		(at 115.57 25.4)
+		(size 58.42 44.45)
+		(fields_autoplaced yes)
+		(stroke
+			(width 0.1524)
+			(type solid)
+		)
+		(fill
+			(color 0 0 0 0.0000)
+		)
+		(property "Sheetname" "Switches, Buttons, LED"
+			(at 115.57 24.6884 0)
+			(effects
+				(font
+					(size 1.27 1.27)
+				)
+				(justify left bottom)
+			)
+		)
+		(property "Sheetfile" "switchesButtonsLed.kicad_sch"
+			(at 115.57 70.4346 0)
+			(effects
+				(font
+					(size 1.27 1.27)
+				)
+				(justify left top)
+			)
+		)
+		(instances
+			(project "pedal_kicad"
+				(path "/bd4452a8-79f4-4b4d-9e93-32f91c7e59e8"
+					(page "3")
+				)
+			)
+		)
+	)
 	(sheet
 		(at 13.97 21.59)

Commit message: commit
Other:
- sheet power_supply ports: added power_supply; removed none
Changed lines of the file:
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@@
+			)
+		)
+		(pin "power_supply" output
+			(at 76.2 76.2 0)
+			(effects
+				(font
+					(size 1.27 1.27)
+				)
+				(justify right)
 			)
 		)
