File: kicad/power_supply.kicad_sch (KiCad schematic)
At the start: 9 parts

Commit message: power suply done
Parts:
- added C16: 4.7u, symbol Device:C
- added R3, R4: 300, symbol Device:R
- added TP1, TP2, TP3, TP5: 3V3 TP, symbol Connector:TestPoint
- renumbered TP1 to TP4
Connections:
- net +5VA: now also R4.1, TP1.1
- net GND: now also C16.2, R3.2, TP5.1
- new net: C16.1, R3.1, R4.2, TP3.1
Other:
- moved on the sheet: C1, C2, C3, C4, C5, C6, R1, R2, TP4

Commit message: commit a crime
Parts:
- removed TP2: 3V3 TP, symbol Connector:TestPoint
- R3: value 300 -> 50k
- R4: value 300 -> 100k
- TP1: renamed from TP5; value 3V3 TP -> GND TP
- TP2: renamed from TP3; value 3V3 TP -> 1V6 TP
- TP3: renamed from TP1; value 3V3 TP -> 5V TP
Connections:
- net +1V5: now reaches C16.1, R3.1, R4.2, TP2.1
Changed lines of the file:
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@@
+	(wire
+		(pts
+			(xy 140.97 86.36) (xy 140.97 87.63)
+		)
+		(stroke
+			(width 0)
+			(type default)
+		)
+	)
 	(wire
 		(pts
@@
 		)
 	)
+	(hierarchical_label "power_supply"
+		(shape input)
+		(at 119.38 58.42 0)
+		(fields_autoplaced yes)
+		(effects
+			(font
+				(size 1.27 1.27)
+			)
+			(justify left)
+		)
+	)
 	(symbol
 		(lib_id "power:GND")
@@
 	)
 	(symbol
+		(lib_id "power:+5VA")
+		(at 140.97 86.36 0)
+		(unit 1)
+		(exclude_from_sim no)
+		(in_bom yes)
+		(on_board yes)
+		(dnp no)
+		(fields_autoplaced yes)
+		(property "Reference" "#PWR014"
+			(at 140.97 90.17 0)
+			(effects
+				(font
+					(size 1.27 1.27)
+				)
+				(hide yes)
+			)
+		)
+		(property "Value" "+1V5"
+			(at 140.97 81.28 0)
+			(effects
+				(font
+					(size 1.27 1.27)
+				)
+			)
+		)
+		(property "Footprint" ""
+			(at 140.97 86.36 0)
+			(effects
+				(font
+					(size 1.27 1.27)
+				)
+				(hide yes)
+			)
+		)
+		(property "Datasheet" ""
+			(at 140.97 86.36 0)
+			(effects
+				(font
+					(size 1.27 1.27)
+				)
+				(hide yes)
+			)
+		)
+		(property "Description" "Power symbol creates a global label with name \"+5VA\""
+			(at 140.97 86.36 0)
+			(effects
+				(font
+					(size 1.27 1.27)
+				)
+				(hide yes)
+			)
+		)
+		(pin "1"
+		)
+		(instances
+			(project "pedal_kicad"
+				(path "/bd4452a8-79f4-4b4d-9e93-32f91c7e59e8/483bf78b-dfb8-4148-a581-618010db7df4"
+					(reference "#PWR014")
+					(unit 1)
+				)
+			)
+		)
+	)
+	(symbol
 		(lib_id "Device:C")
 		(at 86.36 67.31 0)
@@
 		(dnp no)
 		(fields_autoplaced yes)
-		(property "Reference" "TP5"
+		(property "Reference" "TP1"
 			(at 151.13 96.5199 90)
 			(effects
@@
 			)
 		)
-		(property "Value" "3V3 TP"
+		(property "Value" "GND TP"
 			(at 151.13 99.0599 90)
 			(effects
@@
 			(project "pedal_kicad"
 				(path "/bd4452a8-79f4-4b4d-9e93-32f91c7e59e8/483bf78b-dfb8-4148-a581-618010db7df4"
-					(reference "TP5")
+					(reference "TP1")
 					(unit 1)
 				)
@@
 		(dnp no)
 		(fields_autoplaced yes)
-		(property "Reference" "TP3"
+		(property "Reference" "TP2"
 			(at 151.13 86.3599 90)
 			(effects
@@
 			)
 		)
-		(property "Value" "3V3 TP"
+		(property "Value" "1V6 TP"
 			(at 151.13 88.8999 90)
 			(effects
@@
 			(project "pedal_kicad"
 				(path "/bd4452a8-79f4-4b4d-9e93-32f91c7e59e8/483bf78b-dfb8-4148-a581-618010db7df4"
-					(reference "TP3")
+					(reference "TP2")
 					(unit 1)
 				)
@@
 			)
 		)
-		(property "Value" "300"
+		(property "Value" "100k"
 			(at 133.35 82.55 90)
 			(effects
@@
 			)
 		)
-		(property "Value" "300"
+		(property "Value" "50k"
 			(at 133.35 92.71 90)
 			(effects
@@
 		(dnp no)
 		(fields_autoplaced yes)
-		(property "Reference" "TP1"
+		(property "Reference" "TP3"
 			(at 151.13 76.1999 90)
 			(effects
@@
 			)
 		)
-		(property "Value" "3V3 TP"
+		(property "Value" "5V TP"
 			(at 151.13 78.7399 90)
 			(effects
@@
 			(project "pedal_kicad"
 				(path "/bd4452a8-79f4-4b4d-9e93-32f91c7e59e8/483bf78b-dfb8-4148-a581-618010db7df4"
-					(reference "TP1")
+					(reference "TP3")
 					(unit 1)
 				)
@@
 					(unit 1)
 				)
-			)
-		)
-	)
-	(symbol
-		(lib_id "Connector:TestPoint")
-		(at 187.96 96.52 270)
-		(unit 1)
-		(exclude_from_sim no)
-		(in_bom yes)
-		(on_board yes)
-		(dnp no)
-		(fields_autoplaced yes)
-		(property "Reference" "TP2"
-			(at 193.04 95.2499 90)
-			(effects
-				(font
-					(size 1.27 1.27)
-				)
-				(justify left)
-			)
-		)
-		(property "Value" "3V3 TP"
-			(at 193.04 97.7899 90)
-			(effects
-				(font
-					(size 1.27 1.27)
-				)
-				(justify left)
-			)
-		)
-		(property "Footprint" ""
-			(at 187.96 101.6 0)
-			(effects
-				(font
-					(size 1.27 1.27)
-				)
-				(hide yes)
-			)
-		)
-		(property "Datasheet" "~"
-			(at 187.96 101.6 0)
-			(effects
-				(font
-					(size 1.27 1.27)
-				)
-				(hide yes)
-			)
-		)
-		(property "Description" "test point"
-			(at 187.96 96.52 0)
-			(effects
-				(font
-					(size 1.27 1.27)
-				)
-				(hide yes)
-			)
-		)
-		(pin "1"
-		)
-		(instances
-			(project "pedal_kicad"
-				(path "/bd4452a8-79f4-4b4d-9e93-32f91c7e59e8/483bf78b-dfb8-4148-a581-618010db7df4"
-					(reference "TP2")
-					(unit 1)
-				)

Commit message: commit
Changed lines of the file:
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@@
 	)
 	(hierarchical_label "power_supply"
-		(shape input)
+		(shape output)
 		(at 119.38 58.42 0)
 		(fields_autoplaced yes)
